File: DIY305-0201/DIY305.kicad_pcb (KiCad board)
At the start: 2 copper layers, 9.8 x 18.5 mm, 38 parts, among them J4 Conn_02x07_Counter_Clockwise

Commit message: Version 2 with panelization and 0402 design
Parts:
- J4: value Conn_02x07_Counter_Clockwise -> (none)
Changed lines of the file:
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@@
     (property "ki_description" "Generic connector, double row, 02x07, counter clockwise pin numbering scheme (similar to DIP package numbering), script generated (kicad-library-utils/schlib/autogen/connector/)")
     (property "ki_keywords" "connector")
-    (attr through_hole)
+    (attr through_hole board_only exclude_from_pos_files exclude_from_bom allow_missing_courtyard)
     (fp_text reference "J4" (at 3.81 -2.33) (layer "F.SilkS") hide
         (effects (font (size 1 1) (thickness 0.15)))
     )
-    (fp_text value "Conn_02x07_Counter_Clockwise" (at 3.81 17.57) (layer "F.Fab") hide
+    (fp_text value "" (at 3.81 17.57) (layer "F.Fab") hide
         (effects (font (size 1 1) (thickness 0.15)))
     )
@@
     (pad "14" thru_hole circle (at 7.62 0) (size 1.2 1.2) (drill 0.6) (layers "*.Cu" "*.Mask")
       (net 11 "C4") (pinfunction "Pin_14") (pintype "passive"))
-    (model "${KICAD6_3DMODEL_DIR}/Package_DIP.3dshapes/DIP-14_W7.62mm.wrl"
-      (offset (xyz 0 0 0))
-      (scale (xyz 1 1 1))
-      (rotate (xyz 0 0 0))
-    )
   )
   (footprint "LED_SMD:LED_0201_0603Metric" (layer "F.Cu")
