File: DIY305-0201/DIY305.kicad_sch (KiCad schematic)
At the start: 37 parts, among them J4 Conn_02x07_Counter_Clockwise

Commit message: Version 2 with panelization and 0402 design
Parts:
- J4: footprint Package_DIP:DIP-14_W7.62mm -> (none)
Changed lines of the file:
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@@
       (effects (font (size 1.27 1.27)))
     )
-    (property "Footprint" "Package_DIP:DIP-14_W7.62mm" (at 46.99 78.74 0)
+    (property "Footprint" "" (at 46.99 78.74 0)
       (effects (font (size 1.27 1.27)) hide)
     )
