File: DIY305-0402-ALT-PANEL/DIY305.kicad_sch (KiCad schematic)
At the start: 38 parts, among them J1 Conn_01x07, J2 Conn_01x07

Commit message: started work on manually paneling the pcb so I can get a more accurate price quote.
Parts:
- added D100, D101, D102, D103, D104, D105, D106, D107, D108, D109, D110, D111, D112, D113, D114, D115, D116, D117, D118, D119, D120, D121, D122, D123, D124, D125, D126, D127, D128, D129, D130, D131, D132, D133, D134, D135, D136, D137, D138, D139, D140, D141, D142, D143, D144, D37, D38, D39, D40, D41, D42, D43, D44, D45, D46, D47, D48, D49, D50, D51, D52, D53, D54, D55, D56, D57, D58, D59, D60, D61, D62, D63, D64, D65, D66, D67, D68, D69, D70, D71, D72, D73, D74, D75, D76, D77, D78, D79, D80, D81, D82, D83, D84, D85, D86, D87, D88, D89, D90, D91, D92, D93, D94, D95, D96, D97, D98, D99: LED, LED_SMD:LED_0402_1005Metric, symbol Device:LED
- added J3, J4, J5, J6, J7, J8: Conn_01x07, Connector_PinHeader_2.54mm:PinHeader_1x07_P2.54mm_Vertical, symbol Connector_Generic:Conn_01x07
Connections:
- net C1: now also D109.2 (A), D110.2 (A), D111.2 (A), D112.2 (A), D113.2 (A), D114.2 (A), D115.2 (A), D37.2 (A), D38.2 (A), D39.2 (A), D40.2 (A), D41.2 (A), D42.2 (A), D43.2 (A), D73.2 (A), D74.2 (A), D75.2 (A), D76.2 (A), D77.2 (A), D78.2 (A), D79.2 (A), J3.5 (Pin_5), J5.5 (Pin_5), J7.5 (Pin_5)
- net C2: now also D117.2 (A), D118.2 (A), D119.2 (A), D120.2 (A), D121.2 (A), D122.2 (A), D123.2 (A), D45.2 (A), D46.2 (A), D47.2 (A), D48.2 (A), D49.2 (A), D50.2 (A), D51.2 (A), D81.2 (A), D82.2 (A), D83.2 (A), D84.2 (A), D85.2 (A), D86.2 (A), D87.2 (A), J3.1 (Pin_1), J5.1 (Pin_1), J7.1 (Pin_1)
- net C3: now also D124.2 (A), D125.2 (A), D126.2 (A), D127.2 (A), D128.2 (A), D129.2 (A), D130.2 (A), D52.2 (A), D53.2 (A), D54.2 (A), D55.2 (A), D56.2 (A), D57.2 (A), D58.2 (A), D88.2 (A), D89.2 (A), D90.2 (A), D91.2 (A), D92.2 (A), D93.2 (A), D94.2 (A), J4.7 (Pin_7), J6.7 (Pin_7), J8.7 (Pin_7)
- net C4: now also D100.2 (A), D101.2 (A), D131.2 (A), D132.2 (A), D133.2 (A), D134.2 (A), D135.2 (A), D136.2 (A), D137.2 (A), D59.2 (A), D60.2 (A), D61.2 (A), D62.2 (A), D63.2 (A), D64.2 (A), D65.2 (A), D95.2 (A), D96.2 (A), D97.2 (A), D98.2 (A), D99.2 (A), J4.1 (Pin_1), J6.1 (Pin_1), J8.1 (Pin_1)
- net C5: now also D102.2 (A), D103.2 (A), D104.2 (A), D105.2 (A), D106.2 (A), D107.2 (A), D108.2 (A), D138.2 (A), D139.2 (A), D140.2 (A), D141.2 (A), D142.2 (A), D143.2 (A), D144.2 (A), D66.2 (A), D67.2 (A), D68.2 (A), D69.2 (A), D70.2 (A), D71.2 (A), D72.2 (A), J4.2 (Pin_2), J6.2 (Pin_2), J8.2 (Pin_2)
- net DP: now also D116.2 (A), D44.2 (A), D80.2 (A), J3.7 (Pin_7), J5.7 (Pin_7), J7.7 (Pin_7)
- net R1: now also D102.1 (K), D109.1 (K), D117.1 (K), D124.1 (K), D131.1 (K), D138.1 (K), D37.1 (K), D45.1 (K), D52.1 (K), D59.1 (K), D66.1 (K), D73.1 (K), D81.1 (K), D88.1 (K), D95.1 (K), J3.2 (Pin_2), J5.2 (Pin_2), J7.2 (Pin_2)
- net R2: now also D103.1 (K), D110.1 (K), D118.1 (K), D125.1 (K), D132.1 (K), D139.1 (K), D38.1 (K), D46.1 (K), D53.1 (K), D60.1 (K), D67.1 (K), D74.1 (K), D82.1 (K), D89.1 (K), D96.1 (K), J4.3 (Pin_3), J6.3 (Pin_3), J8.3 (Pin_3)
- net R3: now also D104.1 (K), D111.1 (K), D119.1 (K), D126.1 (K), D133.1 (K), D140.1 (K), D39.1 (K), D47.1 (K), D54.1 (K), D61.1 (K), D68.1 (K), D75.1 (K), D83.1 (K), D90.1 (K), D97.1 (K), J3.3 (Pin_3), J5.3 (Pin_3), J7.3 (Pin_3)
- net R4: now also D105.1 (K), D112.1 (K), D120.1 (K), D127.1 (K), D134.1 (K), D141.1 (K), D40.1 (K), D48.1 (K), D55.1 (K), D62.1 (K), D69.1 (K), D76.1 (K), D84.1 (K), D91.1 (K), D98.1 (K), J3.4 (Pin_4), J5.4 (Pin_4), J7.4 (Pin_4)
- net R5: now also D106.1 (K), D113.1 (K), D121.1 (K), D128.1 (K), D135.1 (K), D142.1 (K), D41.1 (K), D49.1 (K), D56.1 (K), D63.1 (K), D70.1 (K), D77.1 (K), D85.1 (K), D92.1 (K), D99.1 (K), J4.4 (Pin_4), J6.4 (Pin_4), J8.4 (Pin_4)
- net R6: now also D100.1 (K), D107.1 (K), D114.1 (K), D122.1 (K), D129.1 (K), D136.1 (K), D143.1 (K), D42.1 (K), D50.1 (K), D57.1 (K), D64.1 (K), D71.1 (K), D78.1 (K), D86.1 (K), D93.1 (K), J4.5 (Pin_5), J6.5 (Pin_5), J8.5 (Pin_5)
- net R7: now also D101.1 (K), D108.1 (K), D115.1 (K), D116.1 (K), D123.1 (K), D130.1 (K), D137.1 (K), D144.1 (K), D43.1 (K), D44.1 (K), D51.1 (K), D58.1 (K), D65.1 (K), D72.1 (K), D79.1 (K), D80.1 (K), D87.1 (K), D94.1 (K), J4.6 (Pin_6), J6.6 (Pin_6), J8.6 (Pin_6)
Other:
- moved on the sheet: D1, D10, D11, D12, D13, D14, D15, D16, D17, D18, D19, D2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
