File: DIY305-0402-PANEL/DIY305.kicad_sch (KiCad schematic)
At the start: 152 parts, among them J1 Conn_01x07, J2 Conn_01x07, J3 Conn_01x07, J4 Conn_01x07, J5 Conn_01x07, J6 Conn_01x07, J7 Conn_01x07, J8 Conn_01x07

Commit message: generated panel and production files
Parts:
- removed D100, D101, D102, D103, D104, D105, D106, D107, D108, D109, D110, D111, D112, D113, D114, D115, D116, D117, D118, D119, D120, D121, D122, D123, D124, D125, D126, D127, D128, D129, D130, D131, D132, D133, D134, D135, D136, D137, D138, D139, D140, D141, D142, D143, D144, D37, D38, D39, D40, D41, D42, D43, D44, D45, D46, D47, D48, D49, D50, D51, D52, D53, D54, D55, D56, D57, D58, D59, D60, D61, D62, D63, D64, D65, D66, D67, D68, D69, D70, D71, D72, D73, D74, D75, D76, D77, D78, D79, D80, D81, D82, D83, D84, D85, D86, D87, D88, D89, D90, D91, D92, D93, D94, D95, D96, D97, D98, D99: LED, LED_SMD:LED_0402_1005Metric, symbol Device:LED
- removed J1, J2, J3, J4, J5, J6, J7, J8: Conn_01x07, Connector_PinHeader_2.54mm:PinHeader_1x07_P2.54mm_Vertical, symbol Connector_Generic:Conn_01x07
- added J3: Conn_01x14, Connector_PinHeader_1.00mm:PinHeader_1x14_P1.00mm_Vertical, symbol Connector_Generic:Conn_01x14
Connections:
- net C1: now also J3.5 (Pin_5)
- net C2: now also J3.1 (Pin_1)
- net C3: now also J3.8 (Pin_8)
- net C4: now also J3.14 (Pin_14)
- net C5: now also J3.13 (Pin_13)
- net DP: now also J3.7 (Pin_7)
- net R1: now also J3.2 (Pin_2)
- net R2: now also J3.12 (Pin_12)
- net R3: now also J3.3 (Pin_3)
- net R4: now also J3.4 (Pin_4)
- net R5: now also J3.11 (Pin_11)
- net R6: now also J3.10 (Pin_10)
- net R7: now also J3.9 (Pin_9)
- no-connect marks 0 -> 1
Other:
- moved on the sheet: D1, D10, D11, D12, D13, D14, D15, D16, D17, D18, D19, D2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
